Commit message: still trying to make the hopper work

File: demo_gazebo/models/hopper_v0.urdf (robot description, URDF)
Before this commit: robot hopper, 7 links, 6 joints
Joints:
- joint leg_to_foot: limit lower=-0.7853975 upper=0.7853975 effort=1000 velocity=0.5 -> lower=-0.7853975 upper=0.7853975 effort=1000 velocity=10000
- joint mid_to_mid2: limit lower=-10 upper=1000 effort=10000 velocity=1000 -> lower=-10 upper=1000 effort=10000 velocity=10000
- joint thigh_to_leg: limit lower=0.0 upper=2.617991667 effort=1000 velocity=0.5 -> lower=0.0 upper=2.617991667 effort=1000 velocity=10000
- joint torso_to_thigh: limit lower=0.0 upper=2.617991667 effort=1000 velocity=0.5 -> lower=0.0 upper=2.617991667 effort=1000 velocity=10000
- joint world_to_mid: limit lower=-1 upper=1000 effort=10000 velocity=1000 -> lower=-1 upper=1000 effort=10000 velocity=10000

File: demo_gazebo/models/hopper_v0.urdf.xacro (robot description, xacro)
@@ -35,6 +35,7 @@
   <xacro:property name="foot_orientation" value="0 1.570795 0" />
   <xacro:property name="max_effort" value="1000" />
-  <xacro:property name="spawn_height" value="0.02" />
+  <xacro:property name="spawn_height" value="0.001" />
   <xacro:property name="gear" value="200" />
+  <xacro:property name="friction_coefficient" value="1" />
   <xacro:property name="density" value="1000" /> <!-- water density -->
   <xacro:property name="foot_mass"  value="${foot_radius*foot_radius*3.14159   * foot_length  * density}" />
@@ -91,5 +92,5 @@
     <parent link="world"/>
     <child link="mid"/>
-    <limit effort="10000" lower="-1" upper="1000" velocity="1000"/>
+    <limit effort="10000" lower="-1" upper="1000" velocity="10000"/>
   </joint>
   <joint name="mid_to_mid2" type="prismatic">
@@ -98,5 +99,5 @@
     <parent link="mid"/>
     <child link="mid2"/>
-    <limit effort="10000" lower="-10" upper="1000" velocity="1000"/>
+    <limit effort="10000" lower="-10" upper="1000" velocity="10000"/>
   </joint>
   <joint name="mid2_to_torso" type="continuous">
@@ -133,5 +134,5 @@
     <parent link="torso"/>
     <child link="thigh"/>
-    <limit effort="${max_effort}" lower="0.0" upper="2.617991667" velocity="1000"/>
+    <limit effort="${max_effort}" lower="0.0" upper="2.617991667" velocity="10000"/>
   </joint>
   <transmission name="torso_to_thigh_tran">
@@ -171,5 +172,5 @@
     <child link="leg"/>
     <axis xyz="0 1 0" rpy="0 0 0" />
-    <limit effort="${max_effort}" lower="0.0" upper="2.617991667" velocity="1000"/>
+    <limit effort="${max_effort}" lower="0.0" upper="2.617991667" velocity="10000"/>
   </joint>
   <transmission name="thigh_to_leg_tran">
@@ -183,4 +184,7 @@
   </transmission>
   <link name="foot">
+    <contact> <!-- PyBullet's way of specifying friction -->
+        <lateral_friction value="${friction_coefficient}"/>
+    </contact>
     <visual>
       <origin xyz="${foot_position_x} ${foot_position_y} ${foot_position_z}" rpy="${foot_orientation}" />
@@ -226,6 +230,6 @@
   </link>
   <gazebo reference="foot">
-    <mu1 value="1"/>
-    <mu2 value="1"/>
+    <mu1 value="${friction_coefficient}"/>
+    <mu2 value="${friction_coefficient}"/>
     <material>Gazebo/Grey</material>
   </gazebo>
@@ -235,5 +239,5 @@
     <child link="foot"/>
     <axis xyz="0 1 0" rpy="0 0 0" />
-    <limit effort="${max_effort}" lower="-0.7853975" upper="0.7853975" velocity="1000"/>
+    <limit effort="${max_effort}" lower="-0.7853975" upper="0.7853975" velocity="10000"/>
   </joint>
   <transmission name="leg_to_foot_tran">

Commit message: pybullet+urdf also learns

File: demo_gazebo/models/hopper_v0.urdf (robot description, URDF)
Before this commit: robot hopper, 7 links, 6 joints
Joints:
- removed joint mid2_to_torso
- removed joint mid_to_mid2
- removed joint world_to_mid
- added joint torso_pitch_joint: type continuous, parent mid2, child torso, origin xyz=0.0 0.0 0 rpy=0 0 0, axis 0 1 0
- added joint torso_x_slider: type prismatic, parent world, child mid, origin xyz=0 0 0 rpy=0 0 0, axis 1 0 0, limit lower=-1 upper=1000 effort=10000 velocity=10000
- added joint torso_z_slider: type prismatic, parent mid, child mid2, origin xyz=0 0 1.211 rpy=0 0 0, axis 0 0 1, limit lower=-10 upper=1000 effort=10000 velocity=10000
