Commit message: many improvements

File: lr_gym/models/cartpole_v0.urdf.xacro (robot description, xacro)
@@ -136,3 +136,37 @@
       </actuator>
     </transmission>
+	<link name="camera_link"/>
+  	<joint name="camera_joint" type="fixed">
+		<origin xyz="0 -3 0.25" rpy="0 0 1.5707" />
+		<parent link="foot_link"/>
+		<child link="camera_link"/>
+	</joint>
+	<gazebo reference="camera_link">
+		<self_collide>0</self_collide>
+		<enable_wind>0</enable_wind>
+		<kinematic>0</kinematic>
+		<enable_gravity>false</enable_gravity>
+		<sensor name="camera" type="camera">
+			<camera name="camera">
+				<horizontal_fov>${69.4*3.14159/180}</horizontal_fov>
+				<image>
+					<width>$(arg camera_width)</width>
+					<height>$(arg camera_height)</height>
+					<format>RGB_INT8</format>
+				</image>
+				<clip>
+					<near>0.01</near>
+					<far>100</far>
+				</clip>
+			</camera>
+			<plugin name="camera/camera_controller" filename="libgazebo_ros_camera.so">
+				<cameraName>camera</cameraName>
+				<frameName>camera_optical_frame</frameName>
+				<updateRate>60</updateRate>
+			</plugin>
+			<always_on>true</always_on>
+			<update_rate>60</update_rate>
+			<visualize>0</visualize>
+		</sensor>
+	</gazebo>
 </robot>

File: lr_gym/models/hopper_v1.urdf.xacro (robot description, xacro)
@@ -334,4 +334,4 @@
         <visualize>0</visualize>
     </sensor>
-</gazebo>
+  </gazebo>
 </robot>

Commit message: cartpole randomization

File: lr_gym/models/cartpole_v0.urdf.xacro (robot description, xacro)
@@ -1,10 +1,57 @@
 <?xml version="1.0" encoding="utf-8"  ?>
-<robot name="cartpole_v0">
-	<gazebo>
-        <plugin name="gazebo_ros_control" filename="libgazebo_ros_control.so">
-            <robotNamespace>/cartpole_v0</robotNamespace>
-						<robotParam>/cartpole_v0_robot_description</robotParam>
-        </plugin>
-    </gazebo>
+<robot name="cartpole_v0" xmlns:xacro="http://www.ros.org/wiki/xacro">
+	<xacro:arg name="bar_width" default="0.05" />
+	<xacro:arg name="bar_length" default="0.05" />
+	<xacro:arg name="bar_height" default="0.8" />
+	<xacro:arg name="bar_mass" default="1" />
+	<xacro:arg name="bar_color" default="1 0.5088 0.0468 1" /> <!-- Orange -->
+	<xacro:arg name="base_width" default="0.4" />
+	<xacro:arg name="base_length" default="0.2" />
+	<xacro:arg name="base_height" default="0.2" />
+	<xacro:arg name="base_mass" default="2.5" />
+	<xacro:arg name="base_color" default="0 0 0 1" /> <!-- Black -->
+	<xacro:arg name="rail_color" default="1 1 1 1" /> <!-- White -->
+	<xacro:arg name="rail_width" default="6" />
+	<xacro:arg name="rail_length" default="0.025" />
+	<xacro:arg name="rail_height" default="0.1" />
+	<xacro:arg name="rail_mass" default="5" />
+	<xacro:arg name="hinge_friction" default="0.1" />
+	<xacro:arg name="rail_friction" default="0.0" />
+	<xacro:arg name="rail_x" default="0.0" />
+	<xacro:arg name="rail_y" default="0.0" />
+	<xacro:arg name="rail_z" default="0.0" />
+	<xacro:arg name="rail_roll" default="0.0" />
+	<xacro:arg name="rail_pitch" default="0.0" />
+	<xacro:arg name="rail_yaw" default="0.0" />
+	<xacro:property name="bar_width" default="$(arg bar_width)" />
+	<xacro:property name="bar_length" default="$(arg bar_length)" />
+	<xacro:property name="bar_height" default="$(arg bar_height)" />
+	<xacro:property name="bar_mass" default="$(arg bar_mass)" />
+	<xacro:property name="bar_color" default="$(arg bar_color)" />
+	<xacro:property name="base_width" default="$(arg base_width)" />
+	<xacro:property name="base_length" default="$(arg base_length)" />
+	<xacro:property name="base_height" default="$(arg base_height)" />
+	<xacro:property name="base_mass" default="$(arg base_mass)" />
+	<xacro:property name="base_color" default="$(arg base_color)" />
+	<xacro:property name="rail_color" default="$(arg rail_color)" />
+	<xacro:property name="rail_width" default="$(arg rail_width)" />
+	<xacro:property name="rail_length" default="$(arg rail_length)" />
+	<xacro:property name="rail_height" default="$(arg rail_height)" />
+	<xacro:property name="rail_mass" default="$(arg rail_mass)" />
+	<xacro:property name="hinge_friction" default="$(arg hinge_friction)" />
+	<xacro:property name="rail_friction" default="$(arg rail_friction)" />
+	<xacro:property name="rail_x" default="$(arg rail_x)" />
+	<xacro:property name="rail_y" default="$(arg rail_y)" />
+	<xacro:property name="rail_z" default="$(arg rail_z)" />
+	<xacro:property name="rail_roll" default="$(arg rail_roll)" />
+	<xacro:property name="rail_pitch" default="$(arg rail_pitch)" />
+	<xacro:property name="rail_yaw" default="$(arg rail_yaw)" />
+	<xacro:macro name="box_inertial" params="mass x y z pose_xyz pose_rpy">
+		<inertial>
+			<origin xyz="${pose_xyz}" rpy="${pose_rpy}"/>
+			<mass value="${mass}" />
+			<inertia ixx="${0.083 * mass * (y*y + z*z)}" ixy="0.0" ixz="0.0" iyy="${0.083 * mass * (x*x + z*z)}" iyz="0.0" izz="${0.083 * mass * (x*x + y*y)}"/>
+		</inertial>
+	</xacro:macro>
 	<!-- * * * Link Definitions * * * -->
   	<!-- * * * Define World Link to fix the foot rail to the world * * * -->
@@ -12,95 +59,89 @@
 	<link name="bar_link">
 		<visual>
-			<origin xyz="0 0 0.4" rpy="0 0 0"/>
+			<origin xyz="0 0 ${bar_height/2}" rpy="0 0 0"/>
 			<geometry>
-				<box size="0.05 0.05 0.8"/>
+				<box size="${bar_width} ${bar_length} ${bar_height}"/>
 			</geometry>
-	     	<material name="brown">
-				<color rgba="0.9 0.8 0.6 1.0"/>
-			</material>
 	   </visual>
 		<collision>
-			<origin xyz="0 0 0.4" rpy="0 0 0"/>
+			<origin xyz="0 0 ${bar_height/2}" rpy="0 0 0"/>
 			<geometry>
-				<box size="0.05 0.05 0.8"/>
+				<box size="${bar_width} ${bar_length} ${bar_height}"/>
 			</geometry>
 	   </collision>
-		<inertial>
-		    <origin xyz="0 0 0.4" rpy="0 0 0"/>
-        	<mass value="1"/>
-        	<inertia ixx="0.0535416666667" ixy="0.0" ixz="0.0" iyy="0.0535416666667" iyz="0.0" izz="0.000416666666667"/>
-        </inertial>
+		<xacro:box_inertial mass="${bar_mass}" x="${bar_width}" y="${bar_length}" z="${bar_height}" pose_xyz="0 0 ${bar_height/2}" pose_rpy="0 0 0"/>
 	</link>
 	<gazebo reference="bar_link">
-		<kp>1000.0</kp>
-        <kd>1000.0</kd>
-        <mu1>0.5</mu1>
-        <mu2>0.5</mu2>
-        <material>Gazebo/Orange</material>
+		<visual name="visual">
+			<material>
+			<ambient>$(arg bar_color)</ambient>
+			<diffuse>$(arg bar_color)</diffuse>
+			<!--
+			<specular>1 0 0 1</specular>
+			<emissive>1 0 0 1</emissive>
+			-->
+			</material>
+      	</visual>
     </gazebo>
 	<link name="base_link">
 		<visual>
-			<origin xyz="0 0 0.2" rpy="0 0 0"/>
+			<origin xyz="0 0 ${base_height}" rpy="0 0 0"/>
 			<geometry>
-				<box size="0.4 0.2 0.2"/>
+				<box size="${base_width} ${base_length} ${base_height}"/>
 			</geometry>
-	     	<material name="black">
-				<color rgba="0 0 0 1.0"/>
-			</material>
 	   </visual>
   		<collision>
-			<origin xyz="0 0 0.2" rpy="0 0 0"/>
+			<origin xyz="0 0 ${base_height}" rpy="0 0 0"/>
 			<geometry>
-				<box size="0.4 0.2 0.2"/>
+				<box size="${base_width} ${base_length} ${base_height}"/>
 			</geometry>
 	   </collision>
-  		<inertial>
-		    <origin xyz="0 0 0.2" rpy="0 0 0"/>
-        	<mass value="2.5"/>
-        	<inertia ixx="0.0166666666667" ixy="0.0" ixz="0.0" iyy="0.0416666666667" iyz="0.0" izz="0.0416666666667"/>
-        </inertial>
+		<xacro:box_inertial mass="${base_mass}" x="${base_width}" y="${base_length}" z="${base_height}" pose_xyz="0 0 ${base_height}" pose_rpy="0 0 0"/>
 	</link>
 	<gazebo reference="base_link">
-        <kp>1000.0</kp>
-        <kd>1000.0</kd>
-        <mu1>0.5</mu1>
-        <mu2>0.5</mu2>
-        <material>Gazebo/Black</material>
+		<visual name="visual">
+			<material>
+			<ambient>$(arg base_color)</ambient>
+			<diffuse>$(arg base_color)</diffuse>
+			<!--
+			<specular>1 0 0 1</specular>
+			<emissive>1 0 0 1</emissive>
+			-->
+			</material>
+      	</visual>
     </gazebo>
 	<link name="foot_link">
+		<origin xyz="${rail_x} ${rail_y} ${rail_z}" rpy="${rail_roll} ${rail_pitch} ${rail_yaw}"/>
 		<visual>
-			<origin xyz="0 0 0.05" rpy="0 0 0"/>
+			<origin xyz="0 0 ${rail_height/2}" rpy="0 0 0"/>
 			<geometry>
-				<box size="6 0.025 0.1"/>
+				<box size="${rail_width} ${rail_length} ${rail_height}"/>
 			</geometry>
-	     	<material name="white">
-				<color rgba="1 1 1 1.0"/>
-			</material>
 	   </visual>
   		<collision>
-			<origin xyz="0 0 0.05" rpy="0 0 0"/>
+			<origin xyz="0 0 ${rail_height/2}" rpy="0 0 0"/>
 			<geometry>
-				<box size="6 0.025 0.1"/>
+				<box size="${rail_width} ${rail_length} ${rail_height}"/>
 			</geometry>
 	   </collision>
-	   <inertial>
-		    <origin xyz="0 0 0.05" rpy="0 0 0"/>
-        	<mass value="5"/>
-        	<inertia ixx="0.00442708333333" ixy="0.0" ixz="0.0" iyy="15.0041666667" iyz="0.0" izz="15.0002604167"/>
-        </inertial>
+		<xacro:box_inertial mass="${rail_mass}" x="${rail_width}" y="${rail_length}" z="${rail_height}" pose_xyz="0 0 ${rail_height/2}" pose_rpy="0 0 0"/>
 	</link>
 	<gazebo reference="foot_link">
-        <kp>1000.0</kp>
-        <kd>1000.0</kd>
-        <mu1>0.5</mu1>
-        <mu2>0.5</mu2>
-        <material>Gazebo/White</material>
+		<visual name="visual">
+			<material>
+			<ambient>$(arg rail_color)</ambient>
+			<diffuse>$(arg rail_color)</diffuse>
+			<!--
+			<specular>1 0 0 1</specular>
+			<emissive>1 0 0 1</emissive>
+			-->
+			</material>
+      	</visual>
     </gazebo>
-<!-- * * * Joint Definitions * * * -->
  	<joint name="cartpole_joint" type="revolute">
     	<parent link="base_link"/>
     	<child link="bar_link"/>
     	<origin xyz="0 0 0.32" rpy="0 0 0"/>
-		<dynamics damping="0.0" friction="0.1"/>
+		<dynamics damping="0.0" friction="${hinge_friction}"/>
        	<limit lower="-1.57" upper="1.57" effort="1" velocity="100"/>
         <axis xyz="0 1 0"/>
@@ -109,4 +150,5 @@
     	<parent link="foot_link"/>
     	<child link="base_link"/>
+		<dynamics damping="0.0" friction="${rail_friction}"/>
        	<limit lower="-2.0" upper="2.0" effort="2000000" velocity="100000"/>
 	</joint>
@@ -115,58 +157,3 @@
         <child link="foot_link"/>
     </joint>
-<!-- * * * Transmission Definitions * * * -->
-	<transmission name="pole_joint_trans">
-      <type>transmission_interface/SimpleTransmission</type>
-      <joint name="cartpole_joint">
-        <hardwareInterface>hardware_interface/EffortJointInterface</hardwareInterface>
-      </joint>
-      <actuator name="pole_jointMotor">
-        <hardwareInterface>hardware_interface/EffortJointInterface</hardwareInterface>
-        <mechanicalReduction>1</mechanicalReduction>
-      </actuator>
-    </transmission>
-	<transmission name="foot_joint_trans">
-      <type>transmission_interface/SimpleTransmission</type>
-      <joint name="foot_joint">
-        <hardwareInterface>hardware_interface/EffortJointInterface</hardwareInterface>
-      </joint>
-      <actuator name="foot_jointMotor">
-        <hardwareInterface>hardware_interface/EffortJointInterface</hardwareInterface>
-        <mechanicalReduction>1</mechanicalReduction>
-      </actuator>
-    </transmission>
-	<link name="camera_link"/>
-  	<joint name="camera_joint" type="fixed">
-		<origin xyz="0 -3 0.25" rpy="0 0 1.5707" />
-		<parent link="foot_link"/>
-		<child link="camera_link"/>
-	</joint>
-	<gazebo reference="camera_link">
-		<self_collide>0</self_collide>
-		<enable_wind>0</enable_wind>
-		<kinematic>0</kinematic>
-		<enable_gravity>false</enable_gravity>
-		<sensor name="camera" type="camera">
-			<camera name="camera">
-				<horizontal_fov>${69.4*3.14159/180}</horizontal_fov>
-				<image>
-					<width>$(arg camera_width)</width>
-					<height>$(arg camera_height)</height>
-					<format>RGB_INT8</format>
-				</image>
-				<clip>
-					<near>0.01</near>
-					<far>100</far>
-				</clip>
-			</camera>
-			<plugin name="camera/camera_controller" filename="libgazebo_ros_camera.so">
-				<cameraName>camera</cameraName>
-				<frameName>camera_optical_frame</frameName>
-				<updateRate>60</updateRate>
-			</plugin>
-			<always_on>true</always_on>
-			<update_rate>60</update_rate>
-			<visualize>0</visualize>
-		</sensor>
-	</gazebo>
 </robot>
